File: right_OBC.sch (KiCad schematic (older format))
At the start: 230 parts, among them M1 S25FL256L, M2 S25FL256L, M3 S25FL256L, M4 CY15B102Q, M5 CY15B102Q, M6 CY15B102Q, Q1 TPS22965-Q1, Q2 TPS22965-Q1, Q3 TPS22965-Q1, U1 STM32L496ZGTx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

Commit message: sync with library
Parts:
- ESD1: footprint VST104_footprints:µDFN-14_3.5x1.35mm -> VST104_footprints:uDFN-14_3.5x1.35mm
Changed lines of the file:
@@
 F 0 "ESD2" H 17000 11650 50  0000 C CNN
 F 1 "SP3012-06" H 17000 10850 50  0000 C CNN
-F 2 "VST104_footprints:µDFN-14_3.5x1.35mm" H 16800 10900 50  0001 C CNN
+F 2 "VST104_footprints:uDFN-14_3.5x1.35mm" H 16800 10900 50  0001 C CNN
 F 3 "https://www.mouser.sk/datasheet/2/240/Littelfuse_TVS_Diode_Array_SP3012_Datasheet.pdf-268239.pdf" H 16800 10900 50  0001 C CNN
 	1    16800 10900
@@
 	1    0    0    -1
 $EndComp
+Wire Wire Line
+	10900 8000 11050 8000
 Wire Bus Line
 	14250 5400 14250 6450
@@
 Wire Bus Line
 	13100 7400 14250 7400
-Wire Wire Line
-	10900 8000 11050 8000
 $EndSCHEMATC
