File: board_delta.sch (KiCad schematic (older format))
At the start: 11 parts

Commit message: pinout doc. update
Other:
- note added: "LEFT\nOBC"
- note added: "RIGHT\n OBC"
Changed lines of the file:
@@
 Text Notes 9250 4725 0    65   ~ 13
 Universal SO-24 footprint\n
+Text Notes 5650 2000 0    197  ~ 39
+LEFT\nOBC
+Text Notes 5550 4050 0    197  ~ 39
+RIGHT\n OBC
 $EndSCHEMATC
